File: ESC-Beta/ESC-Beta.sch (EAGLE design)
At the start: 42 parts, among them IC1 IR2302, IC2 IR2302, IC3 IR2302, Q1 FKI06269, Q2 FKI06269, Q3 FKI06269, Q4 FKI06269, Q5 FKI06269, Q6 FKI06269

Commit message: できた
Parts:
- removed JP1: (no value), pinhead:PINHD-1X3
- removed LED1: (no value), led:LED3MM
- removed R13, R14: 1k, rcl:R-EU_0207/10
Connections:
- removed net N$16: LED1.C, R13.2, R14.2
- net !U_SD: now also SV1.6; no longer SV1.2
- net !W_SD: now also SV1.2; no longer SV1.6
- net BLDC_U: no longer JP1.1
- net BLDC_V: no longer JP1.2
- net BLDC_W: no longer JP1.3
- net GND: no longer R13.1, R14.1
- net U_IN: now also SV1.5; no longer SV1.1
- net VDD: no longer LED1.A
- net W_IN: now also SV1.1; no longer SV1.5
Changed lines of the file:
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@@
 <part name="C6" library="rcl" library_urn="urn:adsk.eagle:library:334" deviceset="C-EU" device="050-024X044" package3d_urn="urn:adsk.eagle:package:23643/1" value="0.1μ"/>
 <part name="C7" library="rcl" library_urn="urn:adsk.eagle:library:334" deviceset="CPOL-EU" device="E5-8.5" package3d_urn="urn:adsk.eagle:package:23374/1" value="100μ"/>
-<part name="LED1" library="led" library_urn="urn:adsk.eagle:library:259" deviceset="LED" device="3MM" package3d_urn="urn:adsk.eagle:package:15797/1"/>
-<part name="VDD8" library="supply1" library_urn="urn:adsk.eagle:library:371" deviceset="VDD" device=""/>
-<part name="R13" library="rcl" library_urn="urn:adsk.eagle:library:334" deviceset="R-EU_" device="0207/10" package3d_urn="urn:adsk.eagle:package:23491/2" value="1k"/>
-<part name="R14" library="rcl" library_urn="urn:adsk.eagle:library:334" deviceset="R-EU_" device="0207/10" package3d_urn="urn:adsk.eagle:package:23491/2" value="1k"/>
-<part name="GND13" library="supply1" library_urn="urn:adsk.eagle:library:371" deviceset="GND" device=""/>
 <part name="Q1" library="transistor-power" library_urn="urn:adsk.eagle:library:400" deviceset="IRF3704" device="-H" package3d_urn="urn:adsk.eagle:package:29490/1" value="FKI06269"/>
 <part name="Q2" library="transistor-power" library_urn="urn:adsk.eagle:library:400" deviceset="IRF3704" device="-H" package3d_urn="urn:adsk.eagle:package:29490/1" value="FKI06269"/>
@@
 <part name="H3" library="holes" library_urn="urn:adsk.eagle:library:237" deviceset="MOUNT-HOLE" device="3.2" package3d_urn="urn:adsk.eagle:package:14275/1"/>
 <part name="H4" library="holes" library_urn="urn:adsk.eagle:library:237" deviceset="MOUNT-HOLE" device="3.2" package3d_urn="urn:adsk.eagle:package:14275/1"/>
-<part name="JP1" library="pinhead" library_urn="urn:adsk.eagle:library:325" deviceset="PINHD-1X3" device="" package3d_urn="urn:adsk.eagle:package:22458/2"/>
 </parts>
 <sheets>
@@
 <attribute name="VALUE" x="206.883" y="74.1426" size="1.778" layer="96"/>
 </instance>
-<instance part="LED1" gate="G$1" x="223.52" y="78.74" smashed="yes">
-<attribute name="NAME" x="227.076" y="74.168" size="1.778" layer="95" rot="R90"/>
-<attribute name="VALUE" x="229.235" y="74.168" size="1.778" layer="96" rot="R90"/>
-</instance>
-<instance part="VDD8" gate="G$1" x="223.52" y="86.36" smashed="yes">
-<attribute name="VALUE" x="221.488" y="87.63" size="1.778" layer="96" rot="R180"/>
-</instance>
-<instance part="R13" gate="G$1" x="223.52" y="66.04" smashed="yes" rot="R90">
-<attribute name="NAME" x="226.06" y="66.0146" size="1.778" layer="95"/>
-<attribute name="VALUE" x="226.06" y="63.754" size="1.778" layer="96"/>
-</instance>
-<instance part="R14" gate="G$1" x="233.68" y="66.04" smashed="yes" rot="R90">
-<attribute name="NAME" x="236.22" y="66.0146" size="1.778" layer="95"/>
-<attribute name="VALUE" x="236.22" y="63.754" size="1.778" layer="96"/>
-</instance>
-<instance part="GND13" gate="1" x="223.52" y="55.88" smashed="yes">
-<attribute name="VALUE" x="220.98" y="53.34" size="1.778" layer="96"/>
-</instance>
 <instance part="Q1" gate="G$1" x="99.06" y="144.78" smashed="yes">
 <attribute name="NAME" x="105.41" y="147.32" size="1.778" layer="95"/>
@@
 <attribute name="NAME" x="65.532" y="23.4442" size="1.778" layer="95"/>
 <attribute name="VALUE" x="65.532" y="20.3962" size="1.778" layer="96"/>
-</instance>
-<instance part="JP1" gate="A" x="111.76" y="25.4" smashed="yes" rot="MR0">
-<attribute name="NAME" x="118.11" y="31.115" size="1.778" layer="95" rot="MR0"/>
-<attribute name="VALUE" x="118.11" y="17.78" size="1.778" layer="96" rot="MR0"/>
 </instance>
 </instances>
@@
 <junction x="101.6" y="137.16"/>
 </segment>
-<segment>
-<pinref part="JP1" gate="A" pin="1"/>
-<wire x1="114.3" y1="27.94" x2="134.62" y2="27.94" width="0.1524" layer="91"/>
-<label x="121.92" y="27.94" size="1.778" layer="95"/>
-</segment>
 </net>
 <net name="N$3" class="0">
@@
 <junction x="200.66" y="73.66"/>
 <pinref part="C7" gate="G$1" pin="-"/>
-</segment>
-<segment>
-<pinref part="R14" gate="G$1" pin="1"/>
-<pinref part="R13" gate="G$1" pin="1"/>
-<wire x1="233.68" y1="60.96" x2="223.52" y2="60.96" width="0.1524" layer="91"/>
-<wire x1="223.52" y1="60.96" x2="223.52" y2="58.42" width="0.1524" layer="91"/>
-<junction x="223.52" y="60.96"/>
-<pinref part="GND13" gate="1" pin="GND"/>
 </segment>
 </net>
@@
 <pinref part="C7" gate="G$1" pin="+"/>
 </segment>
-<segment>
-<pinref part="LED1" gate="G$1" pin="A"/>
-<pinref part="VDD8" gate="G$1" pin="VDD"/>
-<wire x1="223.52" y1="81.28" x2="223.52" y2="83.82" width="0.1524" layer="91"/>
-</segment>
 </net>
 <net name="U_IN" class="0">
@@
 </segment>
 <segment>
-<pinref part="SV1" gate="G$1" pin="1"/>
-<wire x1="152.4" y1="78.74" x2="139.7" y2="78.74" width="0.1524" layer="91"/>
-<label x="139.7" y="78.74" size="1.778" layer="95"/>
+<pinref part="SV1" gate="G$1" pin="5"/>
+<wire x1="152.4" y1="73.66" x2="139.7" y2="73.66" width="0.1524" layer="91"/>
+<label x="139.7" y="73.66" size="1.778" layer="95"/>
 </segment>
 </net>
@@
 </segment>
 <segment>
-<pinref part="SV1" gate="G$1" pin="2"/>
-<wire x1="167.64" y1="78.74" x2="180.34" y2="78.74" width="0.1524" layer="91"/>
-<label x="172.72" y="78.74" size="1.778" layer="95"/>
+<pinref part="SV1" gate="G$1" pin="6"/>
+<wire x1="167.64" y1="73.66" x2="180.34" y2="73.66" width="0.1524" layer="91"/>
+<label x="172.72" y="73.66" size="1.778" layer="95"/>
 </segment>
 </net>
@@
 </segment>
 <segment>
-<pinref part="SV1" gate="G$1" pin="5"/>
-<wire x1="152.4" y1="73.66" x2="139.7" y2="73.66" width="0.1524" layer="91"/>
-<label x="139.7" y="73.66" size="1.778" layer="95"/>
+<pinref part="SV1" gate="G$1" pin="1"/>
+<wire x1="152.4" y1="78.74" x2="139.7" y2="78.74" width="0.1524" layer="91"/>
+<label x="139.7" y="78.74" size="1.778" layer="95"/>
 </segment>
 </net>
@@
 </segment>
 <segment>
-<pinref part="SV1" gate="G$1" pin="6"/>
-<wire x1="167.64" y1="73.66" x2="180.34" y2="73.66" width="0.1524" layer="91"/>
-<label x="172.72" y="73.66" size="1.778" layer="95"/>
+<pinref part="SV1" gate="G$1" pin="2"/>
+<wire x1="167.64" y1="78.74" x2="180.34" y2="78.74" width="0.1524" layer="91"/>
+<label x="172.72" y="78.74" size="1.778" layer="95"/>
 </segment>
 </net>
@@
 <junction x="215.9" y="137.16"/>
 </segment>
-<segment>
-<pinref part="JP1" gate="A" pin="2"/>
-<wire x1="114.3" y1="25.4" x2="134.62" y2="25.4" width="0.1524" layer="91"/>
-<label x="121.92" y="25.4" size="1.778" layer="95"/>
-</segment>
 </net>
 <net name="BLDC_W" class="0">
@@
 <junction x="101.6" y="73.66"/>
 </segment>
-<segment>
-<pinref part="JP1" gate="A" pin="3"/>
-<wire x1="114.3" y1="22.86" x2="134.62" y2="22.86" width="0.1524" layer="91"/>
-<label x="121.92" y="22.86" size="1.778" layer="95"/>
-</segment>
-</net>
-<net name="N$16" class="0">
-<segment>
-<pinref part="R13" gate="G$1" pin="2"/>
-<pinref part="LED1" gate="G$1" pin="C"/>
-<wire x1="223.52" y1="71.12" x2="223.52" y2="73.66" width="0.1524" layer="91"/>
-<pinref part="R14" gate="G$1" pin="2"/>
-<wire x1="233.68" y1="71.12" x2="223.52" y2="71.12" width="0.1524" layer="91"/>
-<junction x="223.52" y="71.12"/>
-</segment>
-</net>
+</net>
